File: PCB/interconnect/MCUs.kicad_sch (KiCad schematic)
At the start: 5 parts, among them J301 Conn_01x15, J302 Conn_01x15

Commit message: PCB Rev 1
Connections:
- no-connect marks 0 -> 15
Changed lines of the file:
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@@
 		(color 0 0 0 0)
 	)
+	(no_connect
+		(at 62.23 45.72)
+	)
+	(no_connect
+		(at 85.09 48.26)
+	)
+	(no_connect
+		(at 62.23 48.26)
+	)
+	(no_connect
+		(at 62.23 53.34)
+	)
+	(no_connect
+		(at 62.23 50.8)
+	)
+	(no_connect
+		(at 85.09 63.5)
+	)
+	(no_connect
+		(at 85.09 66.04)
+	)
+	(no_connect
+		(at 85.09 50.8)
+	)
+	(no_connect
+		(at 62.23 43.18)
+	)
+	(no_connect
+		(at 85.09 71.12)
+	)
+	(no_connect
+		(at 85.09 60.96)
+	)
+	(no_connect
+		(at 85.09 55.88)
+	)
+	(no_connect
+		(at 85.09 68.58)
+	)
+	(no_connect
+		(at 85.09 58.42)
+	)
+	(no_connect
+		(at 62.23 78.74)
+	)
 	(bus_entry
 		(at 275.59 21.59)
@@
 	(wire
 		(pts
+			(xy 264.16 69.85) (xy 273.05 69.85)
+		)
+		(stroke
+			(width 0)
+			(type default)
+		)
+	)
+	(wire
+		(pts
+			(xy 252.73 57.15) (xy 273.05 57.15)
+		)
+		(stroke
+			(width 0)
+			(type default)
+		)
+	)
+	(wire
+		(pts
 			(xy 241.3 35.56) (xy 273.05 35.56)
 		)
@@
 		)
 	)
+	(wire
+		(pts
+			(xy 252.73 62.23) (xy 273.05 62.23)
+		)
+		(stroke
+			(width 0)
+			(type default)
+		)
+	)
 	(bus
 		(pts
@@
 	(wire
 		(pts
+			(xy 252.73 59.69) (xy 273.05 59.69)
+		)
+		(stroke
+			(width 0)
+			(type default)
+		)
+	)
+	(wire
+		(pts
 			(xy 199.39 82.55) (xy 204.47 82.55)
 		)
@@
 		)
 	)
+	(wire
+		(pts
+			(xy 264.16 72.39) (xy 273.05 72.39)
+		)
+		(stroke
+			(width 0)
+			(type default)
+		)
+	)
 	(bus
 		(pts
@@
 	)
 	(label "XIAO.SDA"
-		(at 273.05 69.85 180)
+		(at 264.16 69.85 0)
 		(effects
 			(font
 				(size 1.27 1.27)
 			)
-			(justify right bottom)
+			(justify left bottom)
 		)
 	)
 	(label "ESP32_D32"
-		(at 241.3 35.56 180)
+		(at 241.3 38.1 180)
 		(effects
 			(font
@@
 	)
 	(label "ESP32_D33"
-		(at 241.3 38.1 180)
+		(at 241.3 35.56 180)
 		(effects
 			(font
@@
 	)
 	(label "XIAO.SCL"
-		(at 273.05 72.39 180)
+		(at 264.16 72.39 0)
 		(effects
 			(font
 				(size 1.27 1.27)
 			)
-			(justify right bottom)
+			(justify left bottom)
 		)
 	)
@@
 		)
 	)
-	(label "ESP32_D12"
-		(at 241.3 21.59 180)
-		(effects
-			(font
-				(size 1.27 1.27)
-			)
-			(justify right bottom)
-		)
-	)
 	(label "ULTRASONICS.US1_TRIGG"
 		(at 267.97 21.59 180)
@@
 		)
 	)
+	(label "ESP32_D14"
+		(at 252.73 62.23 180)
+		(effects
+			(font
+				(size 1.27 1.27)
+			)
+			(justify right bottom)
+		)
+	)
 	(label "ESP32_EN"
 		(at 62.23 43.18 180)
@@
 		)
 	)
+	(label "ESP32_D23"
+		(at 252.73 57.15 180)
+		(effects
+			(font
+				(size 1.27 1.27)
+			)
+			(justify right bottom)
+		)
+	)
 	(label "ESP32_RX0"
 		(at 85.09 50.8 0)
@@
 	)
 	(label "ESP32_D25"
-		(at 241.3 29.21 180)
+		(at 241.3 31.75 180)
 		(effects
 			(font
@@
 		)
 	)
-	(label "ESP32_D13"
-		(at 241.3 24.13 180)
-		(effects
-			(font
-				(size 1.27 1.27)
-			)
-			(justify right bottom)
-		)
-	)
 	(label "ESP32_D27"
 		(at 62.23 66.04 180)
@@
 		)
 	)
+	(label "ESP32_D27"
+		(at 252.73 59.69 180)
+		(effects
+			(font
+				(size 1.27 1.27)
+			)
+			(justify right bottom)
+		)
+	)
 	(label "ESP32_D35"
 		(at 62.23 53.34 180)
@@
 		)
 	)
+	(label "ESP32_D12"
+		(at 241.3 24.13 180)
+		(effects
+			(font
+				(size 1.27 1.27)
+			)
+			(justify right bottom)
+		)
+	)
+	(label "ESP32_D13"
+		(at 241.3 21.59 180)
+		(effects
+			(font
+				(size 1.27 1.27)
+			)
+			(justify right bottom)
+		)
+	)
 	(label "ESP32_D26"
-		(at 241.3 31.75 180)
+		(at 241.3 29.21 180)
 		(effects
 			(font

Commit message: Order
Parts:
- J301, J302: now not fitted
Changed lines of the file:
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@@
 		(in_bom yes)
 		(on_board yes)
-		(dnp no)
+		(dnp yes)
 		(property "Reference" "J302"
 			(at 83.566 81.534 0)
@@
 		(in_bom yes)
 		(on_board yes)
-		(dnp no)
+		(dnp yes)
 		(property "Reference" "J301"
 			(at 63.754 81.534 0)

Commit message: Updated PCB, working inference
Parts:
- C302: footprint PCM_JLCPCB:C_0805 -> Capacitor_THT:C_Disc_D5.0mm_W2.5mm_P2.50mm
- R301, R302: footprint PCM_JLCPCB:R_0805 -> PCM_JLCPCB:R_1206
Changed lines of the file:
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@@
 			)
 		)
-		(property "Footprint" "PCM_JLCPCB:R_0805"
+		(property "Footprint" "PCM_JLCPCB:R_1206"
 			(at 192.532 87.63 90)
 			(effects
@@
 			)
 		)
-		(property "Footprint" "PCM_JLCPCB:R_0805"
+		(property "Footprint" "PCM_JLCPCB:R_1206"
 			(at 202.692 87.63 90)
 			(effects
@@
 			)
 		)
-		(property "Footprint" "PCM_JLCPCB:C_0805"
+		(property "Footprint" "Capacitor_THT:C_Disc_D5.0mm_W2.5mm_P2.50mm"
 			(at 106.172 78.74 90)
 			(effects
