File: PCB/interconnect/Ultrasonic.kicad_sch (KiCad schematic)
At the start: 2 parts, among them J701 Conn_01x04

Commit message: Order
Parts:
- J701: now not fitted
- renumbered C501 to C701
Changed lines of the file:
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@@
 		(in_bom yes)
 		(on_board yes)
-		(dnp no)
+		(dnp yes)
 		(fields_autoplaced yes)
 		(property "Reference" "J701"
@@
 		(dnp no)
 		(fields_autoplaced yes)
-		(property "Reference" "#PWR0501"
+		(property "Reference" "#PWR0701"
 			(at 116.84 97.79 0)
 			(effects
@@
 		(dnp no)
 		(fields_autoplaced yes)
-		(property "Reference" "C501"
+		(property "Reference" "C701"
 			(at 119.38 96.5199 0)
 			(effects
@@
 		(dnp no)
 		(fields_autoplaced yes)
-		(property "Reference" "#PWR0502"
+		(property "Reference" "#PWR0702"
 			(at 116.84 110.49 0)
 			(effects

Commit message: Updated PCB, working inference
Parts:
- C701: footprint PCM_JLCPCB:C_0805 -> Capacitor_THT:C_Disc_D5.0mm_W2.5mm_P2.50mm
Changed lines of the file:
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@@
 			)
 		)
-		(property "Footprint" "PCM_JLCPCB:C_0805"
+		(property "Footprint" "Capacitor_THT:C_Disc_D5.0mm_W2.5mm_P2.50mm"
 			(at 115.062 99.06 90)
 			(effects
